File: powermetering.kicad_pcb (KiCad board)
At the start: 2 copper layers, 212 x 103 mm, 215 parts, among them J1 Conn_01x04, J2 Conn_01x02, J3 Conn_01x02, J4 Conn_01x02, J5 Conn_01x02, P1 USB_OTG, P2 CONN_01X04, U1 KSZ8081, U2 ADE9000, U3 STM32F407VETx, U4 USBLC6-4SC6, U5 ACT4088, U6 LNK304D, Y1 Crystal, Y2 25M

Commit message: Change to bigger housing
Parts:
- added D18: ABS2, Diode_SMD:Diode_Bridge_Diotec_ABS, F.Cu at (-73.7, 127.0)
- added D19: ABS2, Diode_SMD:Diode_Bridge_Diotec_ABS, F.Cu at (-65.2, 127.0)
- added T1: Transformer_1P_1S, Transformer_THT:Transformer_CHK_EI30-2VA_1xSec, F.Cu at (111.9, 226.5)
- added T2: Transformer_1P_1S, Transformer_THT:Transformer_CHK_EI30-2VA_1xSec, F.Cu at (140.4, 226.5)
- added T3: Transformer_1P_1S, Transformer_THT:Transformer_CHK_EI30-2VA_1xSec, F.Cu at (169.0, 226.5)
- added U7: LTC4055, Package_DFN_QFN:QFN-16-1EP_4x4mm_P0.65mm_EP2.15x2.15mm, F.Cu at (-34.7, 134.0)
- F1, F2, F3, F4: footprint Fuse:Fuse_2920_7451Metric -> Fuse:Fuseholder_Cylinder-6.3x32mm_Schurter_0031-8002_Horizontal_Open
- J1: footprint TerminalBlock_WAGO:TerminalBlock_WAGO-236_2Stift_RM5mm_4pol -> TerminalBlock_Phoenix:TerminalBlock_Phoenix_PT-1,5-4-5.0-H_1x04_P5.00mm_Horizontal
- J2, J3, J4, J5: footprint TerminalBlock_WAGO:TerminalBlock_WAGO-236_2Stift_RM5mm_2pol -> TerminalBlock_Phoenix:TerminalBlock_Phoenix_PT-1,5-2-5.0-H_1x02_P5.00mm_Horizontal
- moved H12 401.7 mm to (-63.9, 126.8)
- moved H16 393.8 mm to (-56.0, 126.8)
- moved H10 336.3 mm to (-73.9, 134.2)
- moved H14 330.1 mm to (-66.0, 134.2)
- moved H1 301.1 mm to (-48.4, 126.5)
- moved H4 294.0 mm to (-41.4, 134.4)
- moved H2 293.3 mm to (-41.3, 126.5)
- moved H3 286.4 mm to (-34.1, 126.5)
- moved D31 169.0 mm to (234.7, 222.1)
- moved JP1 169.0 mm to (240.1, 211.5)
- moved R65 169.0 mm to (235.2, 211.8)
- moved C50 169.0 mm to (237.3, 222.7)
- moved C51 169.0 mm to (234.4, 217.9)
- moved C55 169.0 mm to (237.3, 219.1)
- moved R58 169.0 mm to (236.6, 215.4)
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Connections:
- C13 pad 1: /IL1N -> Net-(C13-Pad1)
- C14 pad 2: /IL1P -> Net-(C14-Pad2)
- C15 pad 1: /IL2N -> Net-(C15-Pad1)
- C16 pad 2: /IL2P -> Net-(C16-Pad2)
- C17 pad 1: /IL3N -> Net-(C17-Pad1)
- C18 pad 2: /IL3P -> Net-(C18-Pad2)
- C19 pad 1: /INN -> Net-(C19-Pad1)
- C20 pad 2: /INP -> Net-(C20-Pad2)
- C35 pad 1: VPP -> Net-(C35-Pad1)
- C36 pad 2: GNDPWR -> Net-(C36-Pad2)
- C49 pad 1: GND -> Net-(C49-Pad1)
- C49 pad 2: +3V3 -> Net-(C49-Pad2)
- C50 pad 1: GND -> Net-(C50-Pad1)
- C50 pad 2: +3V3 -> Net-(C50-Pad2)
- C51 pad 1: GND -> Net-(C51-Pad1)
- C51 pad 2: +3V3 -> Net-(C51-Pad2)
- C52 pad 1: GND -> Net-(C52-Pad1)
- C52 pad 2: +3V3 -> Net-(C52-Pad2)
- C53 pad 1: GND -> Net-(C53-Pad1)
- C53 pad 2: +3V3 -> Net-(C53-Pad2)
- C54 pad 1: GND -> Net-(C54-Pad1)
- C54 pad 2: +3V3 -> Net-(C54-Pad2)
- C56 pad 1: GND -> Net-(C56-Pad1)
- C56 pad 2: +3V3 -> Net-(C56-Pad2)
- C57 pad 1: GND -> Net-(C57-Pad1)
- C57 pad 2: +3V3 -> Net-(C57-Pad2)
- C58 pad 1: GND -> Net-(C49-Pad1)
- C58 pad 2: +3V3 -> Net-(C49-Pad2)
- C63 pad 1: VPP -> Net-(C63-Pad1)
- C73 pad 2: GNDPWR -> Net-(C73-Pad2)
- D20 pad 1: VPP -> Net-(D20-Pad1)
- D20 pad 2: GNDPWR -> Net-(D20-Pad2)
- D21 pad 1: VPP -> Net-(D20-Pad1)
- D21 pad 2: GNDPWR -> Net-(D20-Pad2)
- D22 pad 1: VPP -> Net-(D20-Pad1)
- D22 pad 2: GNDPWR -> Net-(D20-Pad2)
- R34 pad 2: Net-(D10-Pad1) -> Net-(R34-Pad2)
- R35 pad 1: Net-(D11-Pad2) -> Net-(R35-Pad1)
- R36 pad 2: Net-(D12-Pad1) -> Net-(R36-Pad2)
- R37 pad 1: Net-(D13-Pad2) -> Net-(R37-Pad1)
- R38 pad 2: Net-(D14-Pad1) -> Net-(R38-Pad2)
- R39 pad 1: Net-(D15-Pad2) -> Net-(R39-Pad1)
- R40 pad 2: Net-(D16-Pad1) -> Net-(R40-Pad2)
- R41 pad 1: Net-(D17-Pad2) -> Net-(R41-Pad1)
- R45 pad 1: VPP -> Net-(R45-Pad1)
- R46 pad 2: GNDPWR -> Net-(R46-Pad2)
- Y1 pad 1: Net-(C1-Pad1) -> Net-(Y1-Pad1)
- Y1 pad 2: Net-(C2-Pad1) -> Net-(Y1-Pad2)
Routing:
- net L3: track 64.3 -> 6.15 mm
- net VPP: track 43.8 -> 0.00 mm
- net L2: track 49.7 -> 6.10 mm
- net L1: track 45.3 -> 6.10 mm
- net GNDPWR: track 34.9 -> 0.00 mm
- net Net-(C35-Pad2): track 30.6 -> 0.00 mm
- net /UL3P: track 44.9 -> 27.6 mm
- net /UL2P: track 36.2 -> 26.7 mm
- net /UL1P: track 44.9 -> 36.6 mm
- net Net-(D10-Pad1): track 43.6 -> 38.5 mm
- net Net-(D16-Pad1): track 43.4 -> 38.4 mm
- net Net-(D14-Pad1): track 43.4 -> 38.4 mm
- net Net-(D12-Pad1): track 43.4 -> 38.4 mm
- net Net-(D17-Pad2): track 43.6 -> 38.6 mm
- net Net-(D11-Pad2): track 43.8 -> 38.7 mm
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Other:
- board size 212 x 103 mm -> 255.7 x 232.3 mm

Commit message: add supply and AFE isolation
Parts:
- removed BT1: Battery_Cell, Battery:BatteryHolder_Keystone_1042_1x18650
- removed C71, C72: 10µ, stmbl:C_0805
- removed D32: SS34A, stmbl:SMA_Standard
- removed D33, D34: ES1J R2, stmbl:SMA_Standard
- removed D35: green, stmbl:LED-0805-SIDE
- removed H1, H2, H3, H4, H5, H6, H7, H8: MountingHole_Pad, MountingHole:MountingHole_3.2mm_M3_DIN965_Pad
- removed L5: 10µH 1A, stmbl:SMD_INDUCTOR_32x25
- removed L6: 1m 250mA, stmbl:NPI31W
- removed R69, R71, R72, R76, R77: 1k, stmbl:R_0603
- removed R70: 51k, stmbl:R_0603
- removed R73: 1.5k, stmbl:R_0603
- removed R74: 15k, stmbl:R_0603
- removed R75: 3.9k, stmbl:R_0603
- removed REF**: Symbol_Highvoltage_Type2_CopperTop_Small, Symbol:Symbol_Highvoltage_Type2_CopperTop_Small
- removed T1, T2, T3: Transformer_1P_1S, Transformer_THT:Transformer_CHK_EI30-2VA_1xSec
- added D23: D, stmbl:SMA_Standard, F.Cu at (153.3, 217.3)
- added D24: D, stmbl:SMA_Standard, F.Cu at (179.4, 229.0)
- added R56: 1k, stmbl:R_0603, F.Cu at (216.3, 252.6)
- added R57: 33k, stmbl:R_0805, F.Cu at (149.8, 209.3)
- added R59: 8.2k, stmbl:R_0805, F.Cu at (141.3, 218.8)
- added R60: 51k, stmbl:R_0805, F.Cu at (141.3, 217.2)
- added R61: 8.2k, stmbl:R_0805, F.Cu at (139.3, 222.1)
- added R62: 0, stmbl:R_0805, F.Cu at (149.8, 207.7)
- added R63: 1.3, stmbl:R_1206, F.Cu at (144.1, 207.6)
- added TR2: 750871110, altair04:750871110, F.Cu at (167.5, 210.6)
- added U8: NXE2S0505MC, Converter_DCDC:Converter_DCDC_muRata_NXE2SxxxxMC_THT, F.Cu at (247.8, 206.8)
- added Y3: RTC, stmbl:Crystal_SMD_0603_4Pads, F.Cu at (199.0, 209.8)
- C1, C10, C11, C12, C13, C14, C15, C16, C17, C18, C19, C2, C20, C21, C22, C23, C24, C25, C26, C27, C28, C29, C3, C30, C31, C32, C33, C34, C4, C5, C6, C7, C8, C9: footprint stmbl-kicad-lib:C_0603 -> stmbl:C_0603
- C59, C67: footprint stmbl:C_0603 -> stmbl:C_0805
- C60: value 100n -> 1n; footprint stmbl:C_0603 -> stmbl:C_0805
- C61: footprint stmbl:C_0603 -> stmbl:C_1206
- C62: value 10µ -> 470n
- C64: value 10µ -> 4.7n
- C65: value 100n -> 470µ; footprint stmbl:C_0603 -> Capacitor_SMD:CP_Elec_8x10
- C66: value 10µ -> 100n
- C68: value 10µ -> 470µ; footprint stmbl:C_0805 -> Capacitor_SMD:CP_Elec_8x10.5
- C69, C70: value 10µ -> C; footprint stmbl:C_0805 -> stmbl:C_0603
- D10, D11, D12, D13, D14, D15, D16, D17, D2, D3, D4, D5, D6, D7, D8, D9: footprint stmbl-kicad-lib:SMA_Standard -> stmbl:SMA_Standard
- D18: value ABS2 -> D; footprint Diode_SMD:Diode_Bridge_Diotec_ABS -> stmbl:SMA_Standard
- D19: value ABS2 -> 1.5KExxA; footprint Diode_SMD:Diode_Bridge_Diotec_ABS -> stmbl:SMA_Standard
- D22: footprint Diode_THT:D_DO-201AE_P15.24mm_Horizontal -> stmbl:SMA_Standard
- R68: value 15k -> DNP; footprint stmbl:R_0603 -> stmbl:R_1206
- U5: value ACT4088 -> ALTAIR04-900; footprint stmbl:SOT-23-6 -> Package_SO:SOIC-16_3.9x9.9mm_P1.27mm
- U6: value LNK304D -> AP1117-50; footprint stmbl:SOIC-7 -> Package_TO_SOT_SMD:SOT-223-3_TabPin2
- U7: value LTC4055 -> Si8641ED-B-IS2; footprint Package_DFN_QFN:QFN-16-1EP_4x4mm_P0.65mm_EP2.15x2.15mm -> Package_SO:SOIC-16W_7.5x10.3mm_P1.27mm
- moved H14 341.2 mm to (263.8, 222.0)
- moved U7 276.0 mm to (231.9, 205.5), turned to 90 degrees
- moved C65 261.4 mm to (191.9, 227.6), turned to 270 degrees
- moved H16 257.7 mm to (183.5, 222.0)
- moved C70 255.3 mm to (236.1, 197.9), turned to 90 degrees
- moved C66 250.7 mm to (187.9, 218.4), turned to 180 degrees
- moved C69 249.8 mm to (227.8, 194.5)
- moved C67 248.0 mm to (184.6, 212.2), turned to 90 degrees
- moved H12 247.5 mm to (183.5, 131.6)
- moved C68 241.7 mm to (190.7, 204.6), turned to 180 degrees
- moved D19 240.5 mm to (155.3, 223.1)
- moved C60 235.7 mm to (142.3, 223.2), turned to 270 degrees
- moved D18 235.1 mm to (148.8, 203.2), turned to 270 degrees
- moved C62 235.1 mm to (141.3, 220.5), turned to 180 degrees
- moved C61 233.6 mm to (141.2, 211.2), turned to 180 degrees
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Connections:
- C35 pad 1: Net-(C35-Pad1) -> VPP
- C36 pad 2: Net-(C36-Pad2) -> GNDPWR
- C49 pad 1: Net-(C49-Pad1) -> GND
- C49 pad 2: Net-(C49-Pad2) -> +3V3
- C50 pad 1: Net-(C50-Pad1) -> GND
- C50 pad 2: Net-(C50-Pad2) -> +3V3
- C51 pad 1: Net-(C51-Pad1) -> GND
- C51 pad 2: Net-(C51-Pad2) -> +3V3
- C52 pad 1: Net-(C52-Pad1) -> GND
- C52 pad 2: Net-(C52-Pad2) -> +3V3
- C53 pad 1: Net-(C53-Pad1) -> GND
- C53 pad 2: Net-(C53-Pad2) -> +3V3
- C54 pad 1: Net-(C54-Pad1) -> GND
- C54 pad 2: Net-(C54-Pad2) -> +3V3
- C56 pad 1: Net-(C56-Pad1) -> GND
- C56 pad 2: Net-(C56-Pad2) -> +3V3
- C57 pad 1: Net-(C57-Pad1) -> GND
- C57 pad 2: Net-(C57-Pad2) -> +3V3
- C58 pad 1: Net-(C49-Pad1) -> GND
- C58 pad 2: Net-(C49-Pad2) -> +3V3
- C59 pad 1: Net-(C59-Pad1) -> /VCC
- C59 pad 2: Net-(C59-Pad2) -> GNDPWR
- C60 pad 1: +3.3VP -> /COMP
- C61 pad 1: +3.3VP -> /VCC
- C62 pad 1: +3.3VP -> /COMP
- C62 pad 2: GNDPWR -> Net-(C62-Pad2)
- C63 pad 1: Net-(C63-Pad1) -> VPP
- C64 pad 1: +3.3VP -> /IREF
- C65 pad 2: Net-(C65-Pad2) -> N
- C66 pad 1: Net-(C66-Pad1) -> N
- C66 pad 2: Net-(C65-Pad2) -> Net-(C65-Pad1)
- C67 pad 1: +15V -> +5V
- C67 pad 2: GNDPWR -> N
- C68 pad 1: +15V -> +5V
- C68 pad 2: GNDPWR -> N
- C69 pad 1: +15V -> N
- C69 pad 2: GNDPWR -> +3.3VA
- C70 pad 1: +15V -> N
- C70 pad 2: GNDPWR -> +3.3VA
- C73 pad 2: Net-(C73-Pad2) -> GNDPWR
- D18 pad 1: /DC+ -> /VCC
- D18 pad 2: /DC- -> Net-(D18-Pad2)
- D19 pad 1: /DC+ -> Net-(D19-Pad1)
- D19 pad 2: /DC- -> VPP
- D20 pad 1: Net-(D20-Pad1) -> VPP
- D20 pad 2: Net-(D20-Pad2) -> GNDPWR
- D21 pad 1: Net-(D20-Pad1) -> VPP
- D21 pad 2: Net-(D20-Pad2) -> GNDPWR
- D22 pad 1: Net-(D20-Pad1) -> VPP
- D22 pad 2: Net-(D20-Pad2) -> GNDPWR
- R45 pad 1: Net-(R45-Pad1) -> VPP
- R46 pad 2: Net-(R46-Pad2) -> GNDPWR
- R68 pad 1: Net-(R68-Pad1) -> /SRC
- R68 pad 2: Net-(R68-Pad2) -> GNDPWR
- U5 pad 1: Net-(C59-Pad2) -> /SRC
- U5 pad 2: +15V -> /SRC
- U5 pad 3: Net-(U5-Pad3) -> /VCC
- U5 pad 4: Net-(R68-Pad1) -> GNDPWR
- U5 pad 5: GNDPWR -> /IREF
- U5 pad 6: Net-(C59-Pad1) -> /FB
- U6 pad 1: Net-(C65-Pad1) -> N
- U6 pad 2: Net-(R71-Pad2) -> +5V
- U7 pad 10: GNDPWR -> Net-(U7-Pad10)
- U7 pad 11: Net-(U7-Pad11) -> Net-(U2-Pad38)
- U7 pad 12: Net-(U7-Pad12) -> Net-(U2-Pad40)
- U7 pad 13: Net-(U7-Pad13) -> Net-(U2-Pad39)
- U7 pad 14: Net-(U7-Pad14) -> Net-(U2-Pad37)
- U7 pad 2: Net-(BT1-Pad1) -> Net-(U7-Pad2)
- U7 pad 4: Net-(U7-Pad1) -> Net-(U7-Pad4)
- U7 pad 8: Net-(U7-Pad8) -> Net-(U7-Pad2)
- U7 pad 9: Net-(U7-Pad9) -> Net-(U7-Pad15)
- Y1 pad 1: Net-(Y1-Pad1) -> Net-(C1-Pad1)
- Y1 pad 2: Net-(Y1-Pad2) -> Net-(C2-Pad1)
Routing:
- net VPP: track 0.00 -> 90.7 mm
- net L1: track 6.10 -> 88.8 mm
- net L2: track 6.10 -> 73.3 mm, vias 1 -> 0
- net GNDPWR: track 0.00 -> 37.0 mm, vias 0 -> 20
- net L3: track 6.15 -> 42.8 mm, vias 1 -> 0
- net /UL1P: track 36.6 -> 69.7 mm
- net /UL2P: track 26.7 -> 55.9 mm
- net Net-(F4-Pad1): track 0.00 -> 26.9 mm
- net Net-(C35-Pad2): track 0.00 -> 26.0 mm, vias 0 -> 2
- net Net-(F1-Pad1): track 0.00 -> 25.2 mm
- net /VCC: track 0.00 -> 21.6 mm, vias 0 -> 2
- net N: track 0.00 -> 20.1 mm, vias 0 -> 77
- net Net-(R57-Pad1): track 0.00 -> 19.5 mm
- net Net-(D24-Pad2): track 0.00 -> 19.2 mm
- net /FB: track 0.00 -> 15.7 mm
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- added copper zone on F.Cu, net /DRN
- added copper zone on B.Cu, net GNDPWR
- added copper zone on F.Cu, net GNDPWR
- added copper zone on B.Cu, net N
- added copper zone on F.Cu, net Net-(C35-Pad2)
Other:
- board size 255.7 x 232.3 mm -> 194 x 114.1 mm
- net class Default: via_dia 0.8 -> 0.6; via_drill 0.4 -> 0.35
- board text added: "L1"
- board text added: "L1,2,3 N"
- board text added: "L2"
- board text added: "L3"
- board text added: "N"
- board text removed: "Pls no touchy!"

Commit message: eth phy
Parts:
- removed R55: 1k, stmbl:R_0603
- added C71: C, stmbl:C_0603, F.Cu at (226.0, 200.0)
- added C72: 100n, stmbl:C_0603, F.Cu at (209.7, 213.1)
- added C74: 100n, stmbl:C_0603, F.Cu at (210.9, 213.1)
- added J6: HY951180A_RJ45, stmbl:HY951180A_RJ45, F.Cu at (203.8, 223.2)
- moved C43 102.3 mm to (329.2, 202.4)
- moved C51 102.3 mm to (315.1, 210.4)
- moved R58 102.3 mm to (317.4, 208.0)
- moved C55 102.3 mm to (318.1, 211.6)
- moved R56 102.3 mm to (303.6, 199.2)
- moved C50 102.3 mm to (318.1, 215.3)
- moved JP1 102.3 mm to (320.8, 204.0)
- moved C53 91.8 mm to (317.0, 192.0)
- moved C56 91.8 mm to (319.3, 192.0)
- moved C58 91.8 mm to (317.0, 188.3)
- moved C47 91.8 mm to (318.7, 195.6)
- moved C48 91.8 mm to (316.4, 195.6)
- moved C49 91.8 mm to (315.5, 188.4)
- moved C46 68.9 mm to (302.1, 205.6)
- moved C44 68.9 mm to (298.1, 207.2)
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Connections:
- C65 pad 2: N -> GND
- C66 pad 1: N -> GND
- C67 pad 2: N -> GND
- C68 pad 2: N -> GND
- D31 pad 1: GND -> Net-(D31-Pad1)
- D31 pad 2: Net-(D31-Pad2) -> +3V3
- R56 pad 1: /stm32/STM_MDIO -> /phy_plug/PHY_MDIO
- R67 pad 1: +3V3 -> Net-(D31-Pad1)
- R67 pad 2: Net-(D31-Pad2) -> GND
- TR2 pad 12: N -> GND
- TR2 pad 14: N -> GND
- U3 pad 16: /stm32/STM_MDC -> /phy_plug/PHY_MDC
- U3 pad 24: /stm32/STM_REFCLK -> /phy_plug/PHY_REFCLK
- U3 pad 25: /stm32/STM_MDIO -> /phy_plug/PHY_MDIO
- U3 pad 32: /stm32/STM_CRS -> /phy_plug/PHY_CRS
- U3 pad 33: /stm32/STM_RXD0 -> /phy_plug/PHY_RXD0
- U3 pad 34: /stm32/STM_RXD1 -> /phy_plug/PHY_RXD1
- U3 pad 48: /stm32/STM_TXEN -> /phy_plug/PHY_TXEN
- U3 pad 51: /stm32/STM_TXD0 -> /phy_plug/PHY_TXD0
- U3 pad 52: /stm32/STM_TXD1 -> /phy_plug/PHY_TXD1
- U3 pad 66: /stm32/STM_MCO1 -> /phy_plug/PHY_XI
- U6 pad 1: N -> GND
- U7 pad 1: Net-(U7-Pad1) -> +3V3
- U7 pad 10: Net-(U7-Pad10) -> +3.3VA
- U7 pad 15: Net-(U7-Pad15) -> N
- U7 pad 16: Net-(U7-Pad16) -> +3.3VA
- U7 pad 2: Net-(U7-Pad2) -> GND
- U7 pad 7: Net-(U7-Pad7) -> +3V3
- U7 pad 8: Net-(U7-Pad2) -> GND
- U7 pad 9: Net-(U7-Pad15) -> N
Routing:
- net /phy_plug/PHY_MDIO: track 0.00 -> 30.0 mm, vias 0 -> 2
- net /phy_plug/PHY_MDC: track 0.00 -> 27.0 mm, vias 0 -> 2
- net /phy_plug/PHY_REFCLK: track 0.00 -> 25.5 mm, vias 0 -> 2
- net /phy_plug/PHY_CRS: track 0.00 -> 24.0 mm
- net /phy_plug/PHY_RXD0: track 0.00 -> 21.5 mm
- net /phy_plug/PHY_RXD1: track 0.00 -> 19.2 mm
- net TX_N: track 0.00 -> 17.7 mm
- net RX_P: track 0.00 -> 17.4 mm
- net TX_P: track 0.00 -> 14.6 mm
- net RX_N: track 0.00 -> 14.4 mm
- net /phy_plug/PHY_XI: track 0.00 -> 14.0 mm
- net /phy_plug/PHY_TXEN: track 0.00 -> 13.2 mm, vias 0 -> 2
- net Net-(C72-Pad1): track 0.00 -> 13.1 mm
- net Net-(C74-Pad1): track 0.00 -> 11.4 mm
- net /phy_plug/PHY_TXD1: track 0.00 -> 10.8 mm
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- added copper zone on F.Cu, net GND
- removed copper zone on B.Cu, net N
Other:
- outline, holes or cut-outs redrawn
- net class phy_stuff added: clearance 0.2, trace_width 0.15, via_dia 0.6, via_drill 0.35
- rule trace_min: 0.2 -> 0.15

Commit message: finish routing of bottom board
Parts:
- removed C50, C58: 100n, stmbl:C_0603
- removed C55: 1n, stmbl:C_0603
- added C75: 470µ, Capacitor_SMD:CP_Elec_8x10.5, F.Cu at (328.1, 131.5)
- added C76: 100n, stmbl:C_0805, F.Cu at (318.5, 122.8)
- added C77: 18p, stmbl:C_0603, F.Cu at (330.1, 147.7)
- added C78: 18p, stmbl:C_0603, F.Cu at (327.0, 147.7)
- added J10: CONN_01X02, stmbl:Pin_Header_Straight_1x02, F.Cu at (297.4, 155.0)
- added J7: CONN_01X02, stmbl:Pin_Header_Straight_1x02, F.Cu at (280.6, 144.5)
- added J8: CONN_01X02, stmbl:Pin_Header_Straight_1x02, F.Cu at (335.5, 130.5)
- added J9: CONN_01X02, stmbl:Pin_Header_Straight_1x02, F.Cu at (267.0, 137.5)
- JP1, R58: moved to B.Cu
- moved Y3 136.0 mm to (329.2, 144.4), turned to 270 degrees
- moved C57 127.3 mm to (317.6, 152.2), turned to 270 degrees
- moved C54 116.5 mm to (312.9, 145.2), turned to 270 degrees
- moved C52 114.6 mm to (299.6, 147.8), turned to 0 degrees
- moved P2 101.5 mm to (291.1, 164.8), turned to 90 degrees
- moved Y2 101.0 mm to (322.5, 144.4), turned to 90 degrees
- moved U4 94.5 mm to (293.8, 161.1), turned to 0 degrees
- moved C70 93.8 mm to (301.8, 130.9)
- moved C1 93.3 mm to (288.1, 131.5)
- moved C10 93.3 mm to (291.2, 124.6)
- moved C11 93.3 mm to (291.2, 122.0)
- moved C12 93.3 mm to (291.2, 119.3)
- moved C14 93.3 mm to (277.7, 113.0)
- moved C16 93.3 mm to (292.7, 113.0)
- moved C18 93.3 mm to (307.7, 113.0)
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Connections:
- net /stm32/STM_CS renamed Net-(U3-Pad93)
- C13 pad 1: Net-(C13-Pad1) -> /IL1N
- C14 pad 2: Net-(C14-Pad2) -> /IL1P
- C15 pad 1: Net-(C15-Pad1) -> /IL2N
- C16 pad 2: Net-(C16-Pad2) -> /IL2P
- C17 pad 1: Net-(C17-Pad1) -> /IL3N
- C18 pad 2: Net-(C18-Pad2) -> /IL3P
- C19 pad 1: Net-(C19-Pad1) -> /INN
- C20 pad 2: Net-(C20-Pad2) -> /INP
- C44 pad 2: Net-(C44-Pad2) -> GND
- C45 pad 2: Net-(C44-Pad2) -> GND
- R34 pad 2: Net-(R34-Pad2) -> Net-(D10-Pad1)
- R35 pad 1: Net-(R35-Pad1) -> Net-(D11-Pad2)
- R36 pad 2: Net-(R36-Pad2) -> Net-(D12-Pad1)
- R37 pad 1: Net-(R37-Pad1) -> Net-(D13-Pad2)
- R38 pad 2: Net-(R38-Pad2) -> Net-(D14-Pad1)
- R39 pad 1: Net-(R39-Pad1) -> Net-(D15-Pad2)
- R40 pad 2: Net-(R40-Pad2) -> Net-(D16-Pad1)
- R41 pad 1: Net-(R41-Pad1) -> Net-(D17-Pad2)
- U3 pad 53: Net-(U3-Pad53) -> SS
- U3 pad 55: Net-(U3-Pad55) -> USART3_TX
- U3 pad 56: Net-(U3-Pad56) -> USART3_RX
- U3 pad 8: Net-(U3-Pad8) -> Net-(C77-Pad1)
- U3 pad 89: /stm32/STM_SPI1SCK -> SCLK
- U3 pad 9: Net-(U3-Pad9) -> Net-(C78-Pad1)
- U3 pad 90: /stm32/STM_SPI1MISO -> MISO
- U3 pad 91: /stm32/STM_SPI1MOSI -> MOSI
- U4 pad 4: SWIO -> SWCLK
- U4 pad 6: SWCLK -> SWIO
- U7 pad 3: Net-(U7-Pad3) -> SS
- U7 pad 4: Net-(U7-Pad4) -> SCLK
- U7 pad 5: Net-(U7-Pad5) -> MOSI
- U7 pad 6: Net-(U7-Pad6) -> MISO
- U8 pad 1: Net-(U8-Pad1) -> GND
- U8 pad 3: Net-(U8-Pad3) -> +3V3
- Y3 pad 1: GND -> Net-(C77-Pad1)
- Y3 pad 2: Net-(U3-Pad54) -> Net-(C78-Pad1)
Routing:
- net +3V3: track 1.20 -> 199.4 mm, vias 0 -> 11
- net +3.3VA: track 2.41 -> 48.2 mm, vias 0 -> 3
- net NRST: track 0.00 -> 31.0 mm, vias 0 -> 1
- net MOSI: track 0.00 -> 30.4 mm, vias 0 -> 2
- net SCLK: track 0.00 -> 29.8 mm, vias 0 -> 2
- net MISO: track 0.00 -> 29.6 mm, vias 0 -> 2
- net N: track 20.1 -> 46.6 mm, vias 77 -> 96
- net +5V: track 0.00 -> 25.7 mm
- net Net-(C77-Pad1): track 0.00 -> 23.7 mm
- net GND: track 0.00 -> 19.9 mm, vias 0 -> 61
- net Net-(C65-Pad1): track 0.00 -> 19.5 mm
- net Net-(C78-Pad1): track 0.00 -> 19.2 mm
- net USB-: track 0.00 -> 19.1 mm
- net USB+: track 0.00 -> 19.0 mm
- net Net-(C44-Pad1): track 0.00 -> 18.9 mm
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- added copper zone on B.Cu, net GND
- added copper zone on B.Cu, net N
Other:
- board text removed: "(8x)"
- board text removed: "104.0000"
- board text removed: "110.0000"
- board text removed: "28.0000"
- board text removed: "65.0000"
- board text removed: "76.0000"
- board text removed: "80.8000"
- board text removed: "95.0000"
- board text removed: "ausbrechbar"
